File: DQ542MA Plasma.brd (EAGLE design)
At the start: 100 x 100 mm, 104 parts, among them IC1 MEGA8-P, J1 USB_B_PTH, Q2 16MHZ, Q5 BC849SMD, X3 Phoenix Pluggable 3.81mm 4 way, X4 Phoenix Pluggable 3.81mm 4 way, X5 Phoenix Pluggable 3.81mm 4 way

Commit message: untested gerbers
Routing:
- net GND: vias 69 -> 71
Other:
- board text added: "PWR"
- board text removed: "PWROUT"
