File: DQ542MA ESP32.brd (EAGLE design)
At the start: 100 x 100 mm, 102 parts, among them IC5 1117-33, J1 USB_B_PTH, Q5 BC849SMD, U2 ESP-WROOM-32NARROW, X3 Phoenix Pluggable 3.81mm 4 way, X4 Phoenix Pluggable 3.81mm 4 way, X5 Phoenix Pluggable 3.81mm 4 way

Commit message: ESP32
Routing:
- net GND: vias 120 -> 119
Changed lines of the file:
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@@
 <layer number="20" name="Dimension" color="15" fill="1" visible="yes" active="yes"/>
 <layer number="21" name="tPlace" color="7" fill="1" visible="yes" active="yes"/>
-<layer number="22" name="bPlace" color="7" fill="1" visible="no" active="yes"/>
+<layer number="22" name="bPlace" color="7" fill="1" visible="yes" active="yes"/>
 <layer number="23" name="tOrigins" color="15" fill="1" visible="yes" active="yes"/>
-<layer number="24" name="bOrigins" color="15" fill="1" visible="no" active="yes"/>
-<layer number="25" name="tNames" color="7" fill="1" visible="no" active="yes"/>
-<layer number="26" name="bNames" color="7" fill="1" visible="no" active="yes"/>
-<layer number="27" name="tValues" color="7" fill="1" visible="no" active="yes"/>
-<layer number="28" name="bValues" color="7" fill="1" visible="no" active="yes"/>
+<layer number="24" name="bOrigins" color="15" fill="1" visible="yes" active="yes"/>
+<layer number="25" name="tNames" color="7" fill="1" visible="yes" active="yes"/>
+<layer number="26" name="bNames" color="7" fill="1" visible="yes" active="yes"/>
+<layer number="27" name="tValues" color="7" fill="1" visible="yes" active="yes"/>
+<layer number="28" name="bValues" color="7" fill="1" visible="yes" active="yes"/>
 <layer number="29" name="tStop" color="7" fill="3" visible="yes" active="yes"/>
-<layer number="30" name="bStop" color="7" fill="6" visible="no" active="yes"/>
+<layer number="30" name="bStop" color="7" fill="6" visible="yes" active="yes"/>
 <layer number="31" name="tCream" color="7" fill="9" visible="no" active="yes"/>
 <layer number="32" name="bCream" color="7" fill="5" visible="no" active="yes"/>
@@
 <layer number="37" name="tTest" color="7" fill="1" visible="no" active="yes"/>
 <layer number="38" name="bTest" color="7" fill="1" visible="no" active="yes"/>
-<layer number="39" name="tKeepout" color="4" fill="11" visible="yes" active="yes"/>
+<layer number="39" name="tKeepout" color="4" fill="11" visible="no" active="yes"/>
 <layer number="40" name="bKeepout" color="1" fill="11" visible="no" active="yes"/>
 <layer number="41" name="tRestrict" color="4" fill="10" visible="no" active="yes"/>
@@
 <layer number="43" name="vRestrict" color="2" fill="10" visible="no" active="yes"/>
 <layer number="44" name="Drills" color="7" fill="1" visible="no" active="yes"/>
-<layer number="45" name="Holes" color="7" fill="1" visible="yes" active="yes"/>
+<layer number="45" name="Holes" color="7" fill="1" visible="no" active="yes"/>
 <layer number="46" name="Milling" color="3" fill="1" visible="no" active="yes"/>
 <layer number="47" name="Measures" color="7" fill="1" visible="no" active="yes"/>
@@
 <layer number="154" name="FabDoc2" color="7" fill="1" visible="no" active="yes"/>
 <layer number="155" name="FabDoc3" color="7" fill="1" visible="no" active="yes"/>
-<layer number="156" name="RXDATA" color="9" fill="1" visible="yes" active="yes"/>
-<layer number="157" name="TXDATA" color="12" fill="1" visible="yes" active="yes"/>
+<layer number="156" name="RXDATA" color="9" fill="1" visible="no" active="yes"/>
+<layer number="157" name="TXDATA" color="12" fill="1" visible="no" active="yes"/>
 <layer number="165" name="TEMPLATE" color="15" fill="6" visible="no" active="yes"/>
 <layer number="188" name="Graphics" color="15" fill="1" visible="no" active="yes"/>
@@
 <text x="40.39" y="7.11" size="1.016" layer="21" ratio="18" rot="R90">220U</text>
 <text x="93.4" y="96.5" size="1.778" layer="21" font="vector" ratio="17" rot="R270" align="center">TOOL</text>
-<wire x1="31" y1="91" x2="31" y2="19" width="4.2" layer="30"/>
+<wire x1="31" y1="91" x2="30.9" y2="20.8" width="4.2" layer="30"/>
 <wire x1="36" y1="91" x2="36" y2="21" width="4.2" layer="30"/>
-<wire x1="36" y1="21" x2="40.2" y2="16.8" width="4.2" layer="30"/>
-<wire x1="40.2" y1="16.8" x2="56.7" y2="16.8" width="4.2" layer="30"/>
-<wire x1="56.7" y1="16.8" x2="61.6" y2="11.9" width="4.2" layer="30"/>
-<wire x1="61.6" y1="11.9" x2="61.6" y2="7.9" width="4.2" layer="30"/>
-<wire x1="51.6" y1="7.9" x2="51.6" y2="11.9" width="4.2" layer="30"/>
-<wire x1="51.6" y1="11.9" x2="38.1" y2="11.9" width="4.2" layer="30"/>
-<wire x1="38.1" y1="11.9" x2="31" y2="19" width="4.2" layer="30"/>
 <text x="16" y="24.9" size="0.8128" layer="21" font="vector" ratio="15" align="center">10U</text>
 <rectangle x1="44" y1="37.1" x2="46" y2="37.9" layer="21"/>
@@
 <wire x1="81.5" y1="60.5" x2="87" y2="60.5" width="0.1524" layer="20"/>
 <wire x1="89" y1="62.5" x2="89" y2="67" width="0.1524" layer="20"/>
+<wire x1="31" y1="90.9" x2="31" y2="93.3" width="4" layer="30"/>
+<wire x1="31" y1="93.3" x2="34.7" y2="97" width="4" layer="30"/>
+<wire x1="34.7" y1="97" x2="50.9" y2="97" width="4" layer="30"/>
+<wire x1="50.9" y1="97" x2="54.4" y2="93.5" width="4" layer="30"/>
+<wire x1="54.4" y1="93.5" x2="54.4" y2="83.3" width="4" layer="30"/>
+<wire x1="25.9" y1="21.1" x2="8" y2="39" width="2" layer="30"/>
+<wire x1="8" y1="39" x2="4.1" y2="39" width="2" layer="30"/>
+<wire x1="21" y1="21.1" x2="6.9" y2="35.2" width="2" layer="30"/>
+<wire x1="6.9" y1="35.2" x2="4.3" y2="35.2" width="2" layer="30"/>
+<wire x1="16.1" y1="20.8" x2="5.5" y2="31.4" width="2" layer="30"/>
+<wire x1="5.5" y1="31.4" x2="4.3" y2="31.4" width="2" layer="30"/>
+<wire x1="10.9" y1="21" x2="4.3" y2="27.6" width="2" layer="30"/>
+<wire x1="4.3" y1="27.6" x2="4.3" y2="27.8" width="2" layer="30"/>
+<wire x1="11.1" y1="55.8" x2="9.7" y2="57.2" width="2" layer="30"/>
+<wire x1="9.7" y1="57.2" x2="4" y2="57.2" width="2" layer="30"/>
+<wire x1="15.8" y1="56" x2="10.9" y2="60.9" width="2" layer="30"/>
+<wire x1="10.9" y1="60.9" x2="4.3" y2="60.9" width="2" layer="30"/>
+<wire x1="21.1" y1="55.8" x2="12.2" y2="64.7" width="2" layer="30"/>
+<wire x1="12.2" y1="64.7" x2="4.3" y2="64.7" width="2" layer="30"/>
+<wire x1="25.9" y1="56.1" x2="13.6" y2="68.4" width="2" layer="30"/>
+<wire x1="13.6" y1="68.4" x2="3.9" y2="68.4" width="2" layer="30"/>
+<wire x1="4.1" y1="86.6" x2="5.1" y2="86.6" width="2" layer="30"/>
+<wire x1="5.1" y1="86.6" x2="8" y2="83.7" width="2" layer="30"/>
+<wire x1="8" y1="83.7" x2="19" y2="83.7" width="2" layer="30"/>
+<wire x1="19" y1="83.7" x2="26.1" y2="90.8" width="2" layer="30"/>
+<wire x1="20.8" y1="90.9" x2="17.3" y2="87.4" width="2" layer="30"/>
+<wire x1="17.3" y1="87.4" x2="9.4" y2="87.4" width="2" layer="30"/>
+<wire x1="9.4" y1="87.4" x2="6.5" y2="90.3" width="2" layer="30"/>
+<wire x1="6.5" y1="90.3" x2="4.4" y2="90.3" width="2" layer="30"/>
+<wire x1="4.3" y1="94.2" x2="7.7" y2="94.2" width="2" layer="30"/>
+<wire x1="7.7" y1="94.2" x2="10.7" y2="91.2" width="2" layer="30"/>
+<wire x1="4.5" y1="97.7" x2="9.3" y2="97.7" width="2" layer="30"/>
+<wire x1="9.3" y1="97.7" x2="15.9" y2="91.1" width="2" layer="30"/>
+<wire x1="15.7" y1="15.4" x2="14.2" y2="15.4" width="2" layer="30"/>
+<wire x1="14.2" y1="15.4" x2="8.3" y2="9.5" width="2" layer="30"/>
+<wire x1="8.3" y1="9.5" x2="4.6" y2="9.5" width="2" layer="30"/>
+<wire x1="4.2" y1="5.5" x2="9.5" y2="5.5" width="2" layer="30"/>
+<wire x1="9.5" y1="5.5" x2="13.3" y2="9.3" width="2" layer="30"/>
+<wire x1="13.3" y1="9.3" x2="29.8" y2="9.3" width="2" layer="30"/>
+<wire x1="15.5" y1="3.4" x2="13.1" y2="3.4" width="2" layer="30"/>
+<wire x1="13.1" y1="3.4" x2="11.7" y2="2" width="2" layer="30"/>
+<wire x1="11.7" y1="2" x2="4.4" y2="2" width="2" layer="30"/>
+<wire x1="4.4" y1="2" x2="4.3" y2="1.9" width="2" layer="30"/>
+<wire x1="36.1" y1="91.1" x2="36.9" y2="91.9" width="4" layer="30"/>
+<wire x1="36.9" y1="91.9" x2="42.2" y2="91.9" width="4" layer="30"/>
+<wire x1="42.2" y1="91.9" x2="44.4" y2="89.7" width="4" layer="30"/>
+<wire x1="44.4" y1="89.7" x2="44.4" y2="83" width="4" layer="30"/>
 </plain>
 <attributes>
@@
 <via x="74.4" y="3.1" extent="1-16" drill="0.35"/>
 <via x="65.1" y="10" extent="1-16" drill="0.35"/>
-<via x="65.7" y="46.5" extent="1-16" drill="0.35"/>
 <via x="58.1" y="51.5" extent="1-16" drill="0.35"/>
 <via x="67.3" y="77.4" extent="1-16" drill="0.35"/>

Commit message: update
Parts:
- removed S1: MOMENTARY-SWITCH-SPST-PTH-6.0MM, SparkFun-Switches:TACTILE_SWITCH_PTH_6.0MM
- added PWR: (no value), led:LED3MM
- added R11: 1K, adafruit:R1206
- added R5, R7, R8, R9: 10k, resistor:R1206
- moved S2 8.70 mm to (80.8, 11.6)
Connections:
- new net N$18: PWR.K, R11.1
- net 3.3V: now also R5.2, R7.2, R8.2, R9.2
- net 5V: now also PWR.A
- net CYCLESTART_39: now also R9.1
- net DOOR_35: now also R7.1
- net FEEDHOLD_36: now also R8.1
- net GND: now also R11.2; no longer S1.1
- net RESET/ABORT_34: now also R5.1
- net X_MIN_2: no longer S1.3
Routing:
- net X_MIN_2: track 120.6 -> 62.3 mm, vias 8 -> 5
- net 5V: track 223.9 -> 272.1 mm, vias 2 -> 7
- net C: track 27.3 -> 54.7 mm
- net 3.3V: track 251.2 -> 268.4 mm
- net NC: track 14.0 -> 28.0 mm
- net DOOR_35: track 87.5 -> 101.4 mm
- net FEEDHOLD_36: track 98.1 -> 111.9 mm
- net NO: track 12.2 -> 24.5 mm
- net RESET/ABORT_34: track 90.5 -> 102.3 mm
- net CYCLESTART_39: track 93.7 -> 105.5 mm
- net 0: track 83.9 -> 75.1 mm
- net N$18: track 0.00 -> 6.10 mm
- net 24V: track 277.5 -> 283.0 mm
- net GND: track 100.7 -> 103.5 mm, vias 119 -> 108
- added copper zone on layer 1, net N$1
- added copper zone on layer 1, net N$12
- added copper zone on layer 1, net N$5
- added copper zone on layer 1, net N$7
Other:
- outline, holes or cut-outs redrawn
- board text added: "CNC CONTROLLER"
- board text added: "Designed by"
- board text added: "POWER"
- board text added: "V1.0"
- board text added: "www.facebook.com/beaufortwestcoza"
- board text removed: "GPIO2/XMIN"
